File: flyingsquirrel/_autosave-flyingsquirrel.kicad_sch (KiCad schematic)
At the start: 10 parts, among them J1 Conn_01x02_Pin, U1 XIAO-MG24-DIP, U2 MCP73831-2-OT

Commit message: add footprints
Parts:
- removed D1: RED, symbol Device:LED
- removed D2: GREEN, symbol Device:LED
- removed R1, R2: 470, symbol Device:R
- C1, C2: footprint (none) -> Capacitor_SMD:C_0805_2012Metric_Pad1.18x1.45mm_HandSolder
- J1: footprint (none) -> Connector_JST:JST_PH_S2B-PH-K_1x02_P2.00mm_Horizontal
- R3: footprint (none) -> Capacitor_SMD:C_0603_1608Metric_Pad1.08x0.95mm_HandSolder
Connections:
- net at C2.1, J1.2 (Pin_2), U2.3 (V_{BAT}): now also U1.2 (PC01/A1/D1)
- net at U2.1 (STAT): now also U1.1 (PC00/A0/D0)
