File: flyingsquirrel/flyingsquirrel.kicad_sch (KiCad schematic)
At the start: 0 parts

Commit message: add footprints
Parts:
- added C1, C2: 10uf, symbol Device:C
- added J1: Conn_01x02_Pin, symbol Connector:Conn_01x02_Pin
- added R3: 1.8k, symbol Device:R
- added U1: XIAO-MG24-DIP, Module:MOUDLE14P-XIAO-DIP-SMD, symbol Seeed:XIAO-MG24-DIP
- added U2: MCP73831-2-OT, Package_TO_SOT_SMD:SOT-23-5, symbol Battery_Management:MCP73831-2-OT
Connections:
- new net: C2.1, J1.2 (Pin_2), U1.2 (PC01/A1/D1), U2.3 (V_{BAT})
- new net: U1.1 (PC00/A0/D0), U2.1 (STAT)
- new net: R3.1, U2.5 (PROG)
- new net +5V: C1.1, U1.14 (VIN), U2.4 (V_{DD})
- new net GND: C1.2, C2.2, J1.1 (Pin_1), R3.2, U1.13 (GND), U2.2 (V_{SS})
